Commit message: Changed gazebo material from DarkGrey to FlatBlack

File: open_manipulator_6dof_description/urdf/open_manipulator_6dof.gazebo.xacro (robot description, xacro)
@@ -10,5 +10,5 @@
       <maxVel>1.0</maxVel>
       <minDepth>0.001</minDepth>
-      <material>Gazebo/DarkGrey</material>
+      <material>Gazebo/FlatBlack</material>
     </gazebo>
   </xacro:macro>

File: open_manipulator_6dof_description/urdf/open_manipulator_6dof_torque.urdf.xacro (robot description, xacro)
@@ -317,5 +317,5 @@
         <mesh filename="package://open_manipulator_6dof_description/meshes/chain_link_grip_l.stl" scale="0.001 0.001 0.001"/>
       </geometry>
-      <material name="grey"/>
+      <material name="black"/>
     </visual>
     <collision>
