Commit message: Added gripper dynamics.

File: open_manipulator_6dof_description/urdf/open_manipulator_6dof.urdf.xacro (robot description, xacro)
@@ -340,4 +340,5 @@
   <!--  Gripper link sub -->
   <link name="gripper_link_sub">
+    <dynamics damping="0.5" friction="0.5"/>
     <visual>
       <origin xyz="0.0 -0.0 0" rpy="0 0 0"/>
@@ -370,4 +371,5 @@
   <!--  Gripper joint sub -->
   <joint name="gripper_sub" type="prismatic">
+    <dynamics damping="0.5" friction="0.5"/>
     <parent link="link7"/>
     <child link="gripper_link_sub"/>

Commit message: Changed manipulator color to black.

File: open_manipulator_6dof_description/urdf/open_manipulator_6dof.urdf.xacro (robot description, xacro)
@@ -35,5 +35,5 @@
         <mesh filename="package://open_manipulator_6dof_description/meshes/chain_link1.stl" scale="0.001 0.001 0.001"/>
       </geometry>
-      <material name="grey"/>
+      <material name="black"/>
     </visual>
     <collision>
@@ -75,5 +75,5 @@
         <mesh filename="package://open_manipulator_6dof_description/meshes/chain_link2.stl" scale="0.001 0.001 0.001"/>
       </geometry>
-      <material name="grey"/>
+      <material name="black"/>
     </visual>
     <collision>
@@ -115,5 +115,5 @@
         <mesh filename="package://open_manipulator_6dof_description/meshes/chain_link3.stl" scale="0.001 0.001 0.001"/>
       </geometry>
-      <material name="grey"/>
+      <material name="black"/>
     </visual>
     <collision>
@@ -155,5 +155,5 @@
         <mesh filename="package://open_manipulator_6dof_description/meshes/chain_link4.stl" scale="0.001 0.001 0.001"/>
       </geometry>
-      <material name="grey"/>
+      <material name="black"/>
     </visual>
     <collision>
@@ -195,5 +195,5 @@
         <mesh filename="package://open_manipulator_6dof_description/meshes/chain_link5.stl" scale="0.001 0.001 0.001"/>
       </geometry>
-      <material name="grey"/>
+      <material name="black"/>
     </visual>
     <collision>
@@ -235,5 +235,5 @@
         <mesh filename="package://open_manipulator_6dof_description/meshes/chain_link6.stl" scale="0.001 0.001 0.001"/>
       </geometry>
-      <material name="grey"/>
+      <material name="black"/>
     </visual>
     <collision>
@@ -275,5 +275,5 @@
         <mesh filename="package://open_manipulator_6dof_description/meshes/chain_link7.stl" scale="0.001 0.001 0.001"/>
       </geometry>
-      <material name="grey"/>
+      <material name="black"/>
     </visual>
     <collision>
@@ -305,5 +305,5 @@
         <mesh filename="package://open_manipulator_6dof_description/meshes/chain_link_grip_l.stl" scale="0.001 0.001 0.001"/>
       </geometry>
-      <material name="grey"/>
+      <material name="black"/>
     </visual>
     <collision>
@@ -346,5 +346,5 @@
         <mesh filename="package://open_manipulator_6dof_description/meshes/chain_link_grip_r.stl" scale="0.001 0.001 0.001"/>
       </geometry>
-      <material name="grey"/>
+      <material name="black"/>
     </visual>
     <collision>

File: open_manipulator_6dof_description/urdf/open_manipulator_6dof_torque.urdf.xacro (robot description, xacro)
@@ -47,5 +47,5 @@
         <mesh filename="package://open_manipulator_6dof_description/meshes/chain_link1.stl" scale="0.001 0.001 0.001"/>
       </geometry>
-      <material name="grey"/>
+      <material name="black"/>
     </visual>
     <collision>
@@ -87,5 +87,5 @@
         <mesh filename="package://open_manipulator_6dof_description/meshes/chain_link2.stl" scale="0.001 0.001 0.001"/>
       </geometry>
-      <material name="grey"/>
+      <material name="black"/>
     </visual>
     <collision>
@@ -127,5 +127,5 @@
         <mesh filename="package://open_manipulator_6dof_description/meshes/chain_link3.stl" scale="0.001 0.001 0.001"/>
       </geometry>
-      <material name="grey"/>
+      <material name="black"/>
     </visual>
     <collision>
@@ -167,5 +167,5 @@
         <mesh filename="package://open_manipulator_6dof_description/meshes/chain_link4.stl" scale="0.001 0.001 0.001"/>
       </geometry>
-      <material name="grey"/>
+      <material name="black"/>
     </visual>
     <collision>
@@ -207,5 +207,5 @@
         <mesh filename="package://open_manipulator_6dof_description/meshes/chain_link5.stl" scale="0.001 0.001 0.001"/>
       </geometry>
-      <material name="grey"/>
+      <material name="black"/>
     </visual>
     <collision>
@@ -247,5 +247,5 @@
         <mesh filename="package://open_manipulator_6dof_description/meshes/chain_link6.stl" scale="0.001 0.001 0.001"/>
       </geometry>
-      <material name="grey"/>
+      <material name="black"/>
     </visual>
     <collision>
@@ -287,5 +287,5 @@
         <mesh filename="package://open_manipulator_6dof_description/meshes/chain_link7.stl" scale="0.001 0.001 0.001"/>
       </geometry>
-      <material name="grey"/>
+      <material name="black"/>
     </visual>
     <collision>
@@ -317,5 +317,5 @@
         <mesh filename="package://open_manipulator_6dof_description/meshes/chain_link_grip_l.stl" scale="0.001 0.001 0.001"/>
       </geometry>
-      <material name="grey"/>
+      <material name="black"/>
     </visual>
     <collision>
@@ -357,5 +357,5 @@
         <mesh filename="package://open_manipulator_6dof_description/meshes/chain_link_grip_r.stl" scale="0.001 0.001 0.001"/>
       </geometry>
-      <material name="grey"/>
+      <material name="black"/>
     </visual>
     <collision>

Commit message: Updated urdf xacro.

File: open_manipulator_6dof_description/urdf/open_manipulator_6dof.urdf.xacro (robot description, xacro)
@@ -57,4 +57,7 @@
                izz="1.9267361e-05" />
     </inertial>
+    <gazebo reference="link1">
+      <material>Gazebo/FlatBlack</material>
+    </gazebo>
   </link>
   <!-- Joint 1 -->
@@ -97,4 +100,7 @@
                izz="1.8850320e-05" />
     </inertial>
+    <gazebo reference="link2">
+      <material>Gazebo/FlatBlack</material>
+    </gazebo>
   </link>
   <!--  Joint 2 -->
@@ -137,4 +143,7 @@
                izz="6.0346498e-05" />
     </inertial>-->
+    <gazebo reference="link3">
+      <material>Gazebo/FlatBlack</material>
+    </gazebo>
   </link>
   <!--  Joint 3 -->
@@ -177,4 +186,7 @@
                izz="2.5155057e-04" />
     </inertial>-->
+    <gazebo reference="link4">
+      <material>Gazebo/FlatBlack</material>
+    </gazebo>
   </link>
   <!--  Joint 4 -->
@@ -217,4 +229,7 @@
                izz="9.3127351e-05" />
     </inertial>-->
+    <gazebo reference="link5">
+      <material>Gazebo/FlatBlack</material>
+    </gazebo>
   </link>
   <!--  Joint 5 -->
@@ -257,4 +272,7 @@
                izz="9.3127351e-05" />
     </inertial>
+    <gazebo reference="link6">
+      <material>Gazebo/FlatBlack</material>
+    </gazebo>
   </link>
   <!--  Joint 6 -->
@@ -297,4 +315,7 @@
                izz="9.3127351e-05" />
     </inertial>
+    <gazebo reference="link7">
+      <material>Gazebo/FlatBlack</material>
+    </gazebo>
   </link>
   <!--  Gripper link -->
@@ -327,4 +348,7 @@
                izz="1.7605306e-05" />
     </inertial>-->
+    <gazebo reference="gripper_link">
+      <material>Gazebo/FlatBlack</material>
+    </gazebo>
   </link>
   <!--  Gripper joint -->
